File: z80bankSwitch.kicad_sch (KiCad schematic)
At the start: 33 parts, among them J1 Altera JTAG 10pin Male Connec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, P1 Conn_02x20_Odd_Even, U1 7400, U2 MCP1700x-300xxTT, U3 Z8400, U4 74LS138, U5 EPM3032A Z80 Bank Switcher, U6 AS6C8008-55ZIN, U7 SST39SF040, Y1 Crystal

Commit message: Add missing component values
Parts:
- C1, C3: value C -> 22p
- C13, C14, C2, C6, C8: value C -> 100n
- R1: value R -> 1M
- R2: value R -> 2k
- R3: value R -> 51
- R4: value R -> 470
- R5, R6, R7, R8: value R -> 10k
- Y1: value Crystal -> 4MHz
Other:
- note added: "Series load to reduce ringing"
Changed lines of the file:
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@@
 		)
 	)
+	(text "Series load to \nreduce ringing"
+		(exclude_from_sim no)
+		(at 78.74 194.818 0)
+		(effects
+			(font
+				(size 1.524 1.524)
+			)
+		)
+	)
 	(text "JTAG Port"
 		(exclude_from_sim no)
@@
 			)
 		)
-		(property "Value" "R"
+		(property "Value" "10k"
 			(at 233.68 261.62 90)
 			(show_name no)
@@
 			)
 		)
-		(property "Value" "C"
+		(property "Value" "100n"
 			(at 41.275 247.65 0)
 			(show_name no)
@@
 			)
 		)
-		(property "Value" "C"
+		(property "Value" "100n"
 			(at 128.905 90.17 0)
 			(show_name no)
@@
 			)
 		)
-		(property "Value" "C"
+		(property "Value" "100n"
 			(at 295.275 142.24 0)
 			(show_name no)
@@
 			)
 		)
-		(property "Value" "C"
+		(property "Value" "100n"
 			(at 292.735 46.99 0)
 			(show_name no)
@@
 			)
 		)
-		(property "Value" "C"
+		(property "Value" "100n"
 			(at 132.715 226.06 0)
 			(show_name no)
@@
 			)
 		)
-		(property "Value" "R"
+		(property "Value" "2k"
 			(at 64.77 212.09 90)
 			(show_name no)
@@
 			)
 		)
-		(property "Value" "C"
+		(property "Value" "22p"
 			(at 65.405 226.06 0)
 			(show_name no)
@@
 			)
 		)
-		(property "Value" "C"
+		(property "Value" "22p"
 			(at 34.925 226.06 0)
 			(show_name no)
@@
 			)
 		)
-		(property "Value" "Crystal"
+		(property "Value" "4MHz"
 			(at 48.26 219.71 0)
 			(show_name no)
@@
 			)
 		)
-		(property "Value" "R"
+		(property "Value" "1M"
 			(at 48.26 195.58 90)
 			(show_name no)
@@
 			)
 		)
-		(property "Value" "R"
+		(property "Value" "51"
 			(at 78.74 201.93 90)
 			(show_name no)
@@
 			)
 		)
-		(property "Value" "R"
+		(property "Value" "10k"
 			(at 226.06 261.62 90)
 			(show_name no)
@@
 			)
 		)
-		(property "Value" "R"
+		(property "Value" "10k"
 			(at 201.93 261.62 90)
 			(show_name no)
@@
 			)
 		)
-		(property "Value" "R"
+		(property "Value" "10k"
 			(at 214.63 261.62 90)
 			(show_name no)
@@
 			)
 		)
-		(property "Value" "R"
+		(property "Value" "470"
 			(at 86.36 58.4199 0)
 			(show_name no)
